File: kmm-pmask-mask/kmm-pmask-mask.kicad_pcb (KiCad board)
At the start: 2 copper layers, 90.4 x 109 mm, 78 parts, among them J1 F31L-1A7H1-11030, U1 MS5611-01BA, U10 MAX30101EFD_T, U11 SHT40-AD1B-R3, U12 SHT40-AD1B-R3, U13 TMP117MAIDRVR, U14 TMP117MAIDRVR, U15 TCA9546APW, U2 MAX30101EFD_T, U3 SHT40-AD1B-R3, U4 TMP117MAIDRVR, U5 MS5611-01BA, U6 MS5611-01BA, U7 MS5611-01BA, U8 MAX30101EFD_T, U9 MAX30101EFD_T

Commit message: minor track tweaks
Routing:
- net +3.3V: track 346.7 -> 347.6 mm, vias 20 -> 19
