File: kmm-pmask-control/MCU.kicad_sch (KiCad schematic)
At the start: 0 parts

Commit message: Initial draft of control board
Parts:
- added C11: 10u, Capacitor_SMD:C_0603_1608Metric_Pad1.08x0.95mm_HandSolder, symbol Device:C
- added C12: 1u, Capacitor_SMD:C_0402_1005Metric_Pad0.74x0.62mm_HandSolder, symbol Device:C
- added C15: 100n, Capacitor_SMD:C_0402_1005Metric_Pad0.74x0.62mm_HandSolder, symbol Device:C
- added D6, D7, D8, D9: LED GREEN, LED_SMD:LED_0603_1608Metric_Pad1.05x0.95mm_HandSolder, symbol Device:LED
- added R12, R13: 4.7k, Resistor_SMD:R_0402_1005Metric_Pad0.72x0.64mm_HandSolder, symbol Device:R
- added R14, R15, R16, R17, R19: 10k, Resistor_SMD:R_0402_1005Metric_Pad0.72x0.64mm_HandSolder, symbol Device:R
- added SW2: EVQ-P2402W, Button_Switch_SMD:SW_SPST_EVQP2_ShortPushTravel_H2.5mm, symbol Switch:SW_SPST
- added TP14: I2C SCL, TestPoint:TestPoint_Pad_D1.5mm, symbol Connector:TestPoint
- added TP15: I2C SDA, TestPoint:TestPoint_Pad_D1.5mm, symbol Connector:TestPoint
- added TP16: I2C EN, TestPoint:TestPoint_Pad_D1.5mm, symbol Connector:TestPoint
- added TP17: I2C RST, TestPoint:TestPoint_Pad_D1.5mm, symbol Connector:TestPoint
- added TP18: GND, TestPoint:TestPoint_Pad_D1.5mm, symbol Connector:TestPoint
- added U5: MDBT50Q-P1MV2, RF_Module:Raytac_MDBT50Q, symbol RF_Module:MDBT50Q-P1MV2
Connections:
- new net: D6.1 (K), R14.1
- new net: D8.1 (K), R16.1
- new net: D7.1 (K), R15.1
- new net: D9.1 (K), R17.1
- new net +3.3V: C11.1, C12.1, D6.2 (A), D7.2 (A), D8.2 (A), D9.2 (A), R12.1, R13.1, R19.1, U5.28 (VDD), U5.30 (VDDH)
- new net BATT_SENSE: U5.12 (P0.31)
- new net DEBUG_LED0: R14.2, U5.42 (P0.19)
- new net DEBUG_LED1: R15.2, U5.44 (P0.20)
- new net DEBUG_LED2: R16.2, U5.43 (P0.21)
- new net DEBUG_LED3: R17.2, U5.46 (P0.22)
- new net GND: C11.2, C12.2, C15.2, SW2.1 (A), TP18.1, U5.1 (GND), U5.15 (GND), U5.2 (GND), U5.33 (GND), U5.55 (GND)
- new net I2C.EN: TP16.1, U5.36 (P0.14)
- new net I2C.SCL: R12.2, TP14.1, U5.37 (P0.13)
- new net I2C.SDA: R13.2, TP15.1, U5.39 (P0.15)
- new net I2C.~{RST}: TP17.1, U5.38 (P0.16)
- new net PRESEN.A: U5.13 (P0.28)
- new net PRESEN.B: U5.14 (P0.30)
- new net SPI.CLK: U5.27 (P0.11)
- new net SPI.CS: U5.23 (P0.07)
- new net SPI.SDI: U5.26 (P1.09)
- new net SPI.SDO: U5.29 (P0.12)
- new net SWD.CLK: U5.53 (SWDCLK)
- new net SWD.IO: U5.51 (SWDIO)
- new net ~{RESET}: C15.1, R19.2, SW2.2 (B), U5.40 (P0.18)
- no-connect marks 0 -> 36
Other:
- note added: "General-Purpose Debug LEDs"
- note added: "Reset Button"
- note added: "Test Points, I2C"
- note added: "nRF52840 SiP"
- title: (none) -> MCU

Commit message: Initial PCB Layout
Parts:
- removed TP17: I2C RST, TestPoint:TestPoint_Pad_D1.5mm, symbol Connector:TestPoint
- TP14, TP15, TP16, TP18: footprint TestPoint:TestPoint_Pad_D1.5mm -> TestPoint:TestPoint_Pad_D1.0mm
Connections:
- net DEBUG_LED1: now also U5.43 (P0.21); no longer U5.44 (P0.20)
- net DEBUG_LED2: now also U5.44 (P0.20); no longer U5.43 (P0.21)
- net I2C.SCL: now also R13.2, U5.39 (P0.15); no longer R12.2, U5.37 (P0.13)
- net I2C.SDA: now also R12.2, U5.37 (P0.13); no longer R13.2, U5.39 (P0.15)
- net PRESEN.A: now also U5.14 (P0.30); no longer U5.13 (P0.28)
- net PRESEN.B: now also U5.13 (P0.28); no longer U5.14 (P0.30)
- net SPI.CS: now also U5.29 (P0.12); no longer U5.23 (P0.07)
- net SPI.SDO: now also U5.23 (P0.07); no longer U5.29 (P0.12)
Changed lines of the file:
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@@
 		)
 	)
-	(bus_entry
-		(at 228.6 107.95)
-		(size 2.54 2.54)
-		(stroke
-			(width 0)
-			(type default)
-		)
-	)
 	(wire
 		(pts
@@
 		)
 	)
-	(bus
-		(pts
-			(xy 228.6 92.71) (xy 228.6 107.95)
-		)
-		(stroke
-			(width 0)
-			(type default)
-		)
-	)
 	(wire
 		(pts
@@
 	(wire
 		(pts
-			(xy 231.14 110.49) (xy 241.3 110.49)
-		)
-		(stroke
-			(width 0)
-			(type default)
-		)
-	)
-	(wire
-		(pts
 			(xy 231.14 95.25) (xy 241.3 95.25)
 		)
@@
 		)
 	)
+	(bus
+		(pts
+			(xy 228.6 92.71) (xy 228.6 102.87)
+		)
+		(stroke
+			(width 0)
+			(type default)
+		)
+	)
 	(wire
 		(pts
@@
 		)
 	)
-	(label "PRESEN.A"
-		(at 55.88 78.74 0)
-		(effects
-			(font
-				(size 1.27 1.27)
-			)
-			(justify left bottom)
-		)
-	)
-	(label "PRESEN.B"
-		(at 55.88 83.82 0)
+	(label "DEBUG_LED1"
+		(at 139.7 106.68 0)
 		(effects
 			(font
@@
 	)
 	(label "SPI.SDO"
-		(at 139.7 129.54 0)
-		(effects
-			(font
-				(size 1.27 1.27)
-			)
-			(justify left bottom)
-		)
-	)
-	(label "I2C.SCL"
-		(at 139.7 81.28 0)
+		(at 139.7 137.16 0)
 		(effects
 			(font
@@
 		)
 	)
-	(label "I2C.~{RST}"
-		(at 241.3 110.49 180)
-		(effects
-			(font
-				(size 1.27 1.27)
-			)
-			(justify right bottom)
-		)
-	)
 	(label "SPI.CS"
-		(at 139.7 137.16 0)
+		(at 139.7 129.54 0)
 		(effects
 			(font
@@
 	)
 	(label "I2C.SDA"
-		(at 139.7 86.36 0)
+		(at 139.7 81.28 0)
 		(effects
 			(font
@@
 		)
 	)
-	(label "DEBUG_LED1"
-		(at 139.7 104.14 0)
+	(label "PRESEN.B"
+		(at 55.88 78.74 0)
 		(effects
 			(font
@@
 		)
 	)
-	(label "SPI.SDI"
-		(at 139.7 134.62 0)
+	(label "DEBUG_LED3"
+		(at 139.7 109.22 0)
 		(effects
 			(font
@@
 		)
 	)
-	(label "DEBUG_LED2"
-		(at 139.7 106.68 0)
+	(label "I2C.SCL"
+		(at 139.7 86.36 0)
 		(effects
 			(font
@@
 		)
 	)
-	(label "SPI.CLK"
-		(at 139.7 132.08 0)
+	(label "PRESEN.A"
+		(at 55.88 83.82 0)
 		(effects
 			(font
@@
 		)
 	)
-	(label "DEBUG_LED3"
-		(at 139.7 109.22 0)
+	(label "SPI.CLK"
+		(at 139.7 132.08 0)
 		(effects
 			(font
@@
 		)
 	)
+	(label "DEBUG_LED2"
+		(at 139.7 104.14 0)
+		(effects
+			(font
+				(size 1.27 1.27)
+			)
+			(justify left bottom)
+		)
+	)
 	(label "DEBUG_LED0"
 		(at 139.7 101.6 0)
@@
 		)
 	)
+	(label "SPI.SDI"
+		(at 139.7 134.62 0)
+		(effects
+			(font
+				(size 1.27 1.27)
+			)
+			(justify left bottom)
+		)
+	)
 	(label "SWD.CLK"
 		(at 54.61 63.5 0)
@@
 			)
 		)
-		(property "Footprint" "TestPoint:TestPoint_Pad_D1.5mm"
+		(property "Footprint" "TestPoint:TestPoint_Pad_D1.0mm"
 			(at 241.3 105.41 0)
 			(hide yes)
@@
 			)
 		)
-		(property "Footprint" "TestPoint:TestPoint_Pad_D1.5mm"
+		(property "Footprint" "TestPoint:TestPoint_Pad_D1.0mm"
 			(at 262.89 102.87 0)
 			(hide yes)
@@
 			)
 		)
-		(property "Footprint" "TestPoint:TestPoint_Pad_D1.5mm"
+		(property "Footprint" "TestPoint:TestPoint_Pad_D1.0mm"
 			(at 241.3 100.33 0)
 			(hide yes)
@@
 	)
 	(symbol
-		(lib_id "Connector:TestPoint")
-		(at 241.3 110.49 270)
-		(unit 1)
-		(body_style 1)
-		(exclude_from_sim no)
-		(in_bom yes)
-		(on_board yes)
-		(in_pos_files yes)
-		(dnp no)
-		(fields_autoplaced yes)
-		(property "Reference" "TP17"
-			(at 246.38 109.2199 90)
-			(show_name no)
-			(do_not_autoplace no)
-			(effects
-				(font
-					(size 1.27 1.27)
-				)
-				(justify left)
-			)
-		)
-		(property "Value" "I2C RST"
-			(at 246.38 111.7599 90)
-			(show_name no)
-			(do_not_autoplace no)
-			(effects
-				(font
-					(size 1.27 1.27)
-				)
-				(justify left)
-			)
-		)
-		(property "Footprint" "TestPoint:TestPoint_Pad_D1.5mm"
-			(at 241.3 115.57 0)
-			(hide yes)
-			(show_name no)
-			(do_not_autoplace no)
-			(effects
-				(font
-					(size 1.27 1.27)
-				)
-			)
-		)
-		(property "Datasheet" ""
-			(at 241.3 115.57 0)
-			(hide yes)
-			(show_name no)
-			(do_not_autoplace no)
-			(effects
-				(font
-					(size 1.27 1.27)
-				)
-			)
-		)
-		(property "Description" "test point"
-			(at 241.3 110.49 0)
-			(hide yes)
-			(show_name no)
-			(do_not_autoplace no)
-			(effects
-				(font
-					(size 1.27 1.27)
-				)
-			)
-		)
-		(pin "1"
-		)
-		(instances
-			(project "kmm-pmask-control"
-				(path "/c80d922d-876d-4b9c-ac92-42497602c2d1/841086c9-4c99-4f37-bfb8-92a537b93af0"
-					(reference "TP17")
-					(unit 1)
-				)
-			)
-		)
-	)
-	(symbol
 		(lib_id "Device:R")
 		(at 220.98 77.47 90)
@@
 			)
 		)
-		(property "Footprint" "TestPoint:TestPoint_Pad_D1.5mm"
+		(property "Footprint" "TestPoint:TestPoint_Pad_D1.0mm"
 			(at 241.3 110.49 0)
 			(hide yes)
