File: kmm-pmask-control/ext_conn.kicad_sch (KiCad schematic)
At the start: 14 parts, among them J1 F31L-1A7H1-11030, U1 PCA9517ADP

Commit message: WIP power circuitry
Other:
- note added: "30 pos 0.5mm pitch Zero Insertion Force"
- note added: "Shorted to GND on slave side"
Changed lines of the file:
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@@
+	)
+	(rectangle
+		(start 71.12 132.08)
+		(end 90.17 139.7)
+		(stroke
+			(width 0)
+			(type default)
+		)
+		(fill
+			(type none)
+		)
 	)
 	(rectangle
@@
 		)
 	)
+	(text "30 pos\n0.5mm pitch\nZero Insertion Force"
+		(exclude_from_sim no)
+		(at 236.855 85.725 0)
+		(effects
+			(font
+				(size 1.27 1.27)
+			)
+			(justify left top)
+		)
+	)
 	(text "Power Output\n5.0V: 1.0A max\n3.3V: 1.0A max\n1.8V: 0.5A max"
 		(exclude_from_sim no)
@@
 			)
 			(justify right)
+		)
+	)
+	(text "Shorted to GND on slave side"
+		(exclude_from_sim no)
+		(at 88.9 146.05 0)
+		(effects
+			(font
+				(size 1.27 1.27)
+			)
+			(justify left top)
 		)
 	)
@@
 		)
 	)
-	(text_box "This part is not strictly nessesary, it is insurance against unforseen extra bus capacitance from the FFC or mask PCB.\nThis targets I2C FM (400 kHz), which has a bus capacitance limit of 400 pF.\n\nA conservative estimate of worst-case bus capacitances across the entire system is as follows:\n	Cable (1m FFC): 40 pF\n	Downstream I2C switch (TCA9546APW): 19 pF (input side) / 6 pF (per channel, 4 channels total)\n		Worst-case devices on one switch channel: 30 pF\n		Worst-case trace capacitance on one switch channel: 50 pF\nWorst-case scenario (All switch channels enabled): 403 pF (already over limit)\n\nAs capacitance estimates are conservative-worst case and there is no reason for all switch channels to be enabled, it is unlikely for the worst-case scenario to occur.\nHowever, this component is included to increase the safety margin should a similar event occur."
+	(text_box "0.33 mA per pin\nwhen connected"
+		(exclude_from_sim no)
+		(at 97.79 121.9978 0)
+		(size 21.59 6.2721)
+		(margins 0.9525 0.9525 0.9525 0.9525)
+		(stroke
+			(width 0)
+			(type solid)
+		)
+		(fill
+			(type none)
+		)
+		(effects
+			(font
+				(size 1.27 1.27)
+			)
+			(justify left top)
+		)
+	)
+	(text_box "This part is not strictly nessesary, it is insurance against unforseen extra bus capacitance from the FFC or mask PCB.\nThis targets I2C FM (400 kHz), which has a bus capacitance limit of 400 pF.\n\nA conservative estimate of worst-case bus capacitances across the downstream system is as follows:\n	Cable (1 m FFC): 40 pF\n	Downstream I2C switch (TCA9546APW): 19 pF (input side) / 6 pF (per channel, 4 channels total)\n		Worst-case devices on one switch channel: 30 pF\n		Worst-case trace capacitance on one switch channel: 50 pF\nWorst-case scenario (All switch channels enabled): 403 pF (already over limit)\n\nAs capacitance estimates are conservative worst-case and there is no reason for all switch channels to be enabled, it is unlikely for the worst-case scenario to occur.\nThis component is included to increase the safety margin should a lesser event occur."
 		(exclude_from_sim no)
 		(at 39.37 83.82 0)
@@
 		)
 		(stroke
+			(width 0)
+			(type default)
+		)
+	)
+	(polyline
+		(pts
+			(xy 90.17 132.08) (xy 97.79 128.27)
+		)
+		(stroke

Commit message: Initial draft of control board
Parts:
- added C13, C14: 100n, Capacitor_SMD:C_0402_1005Metric_Pad0.74x0.62mm_HandSolder, symbol Device:C
Connections:
- net +3.3V: now also C13.1, C14.1
- net GND: now also C13.2, C14.2
Other:
- note added: "Place one cap each for pins 1,8"
- moved on the sheet: J1, R1, R2, R3, U1

Commit message: Initial PCB Layout
Parts:
- TP1, TP2, TP3, TP4, TP5, TP6, TP7: footprint TestPoint:TestPoint_Pad_D1.5mm -> TestPoint:TestPoint_Pad_D1.0mm
Changed lines of the file:
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@@
 			)
 		)
-		(property "Footprint" "TestPoint:TestPoint_Pad_D1.5mm"
+		(property "Footprint" "TestPoint:TestPoint_Pad_D1.0mm"
 			(at 147.32 132.08 0)
 			(hide yes)
@@
 			)
 		)
-		(property "Footprint" "TestPoint:TestPoint_Pad_D1.5mm"
+		(property "Footprint" "TestPoint:TestPoint_Pad_D1.0mm"
 			(at 134.62 158.75 0)
 			(hide yes)
@@
 			)
 		)
-		(property "Footprint" "TestPoint:TestPoint_Pad_D1.5mm"
+		(property "Footprint" "TestPoint:TestPoint_Pad_D1.0mm"
 			(at 147.32 152.4 0)
 			(hide yes)
@@
 			)
 		)
-		(property "Footprint" "TestPoint:TestPoint_Pad_D1.5mm"
+		(property "Footprint" "TestPoint:TestPoint_Pad_D1.0mm"
 			(at 151.13 158.75 0)
 			(hide yes)
@@
 			)
 		)
-		(property "Footprint" "TestPoint:TestPoint_Pad_D1.5mm"
+		(property "Footprint" "TestPoint:TestPoint_Pad_D1.0mm"
 			(at 147.32 137.16 0)
 			(hide yes)
@@
 			)
 		)
-		(property "Footprint" "TestPoint:TestPoint_Pad_D1.5mm"
+		(property "Footprint" "TestPoint:TestPoint_Pad_D1.0mm"
 			(at 147.32 142.24 0)
 			(hide yes)
@@
 			)
 		)
-		(property "Footprint" "TestPoint:TestPoint_Pad_D1.5mm"
+		(property "Footprint" "TestPoint:TestPoint_Pad_D1.0mm"
 			(at 147.32 147.32 0)
 			(hide yes)
