File: kmm-pmask-control/power.kicad_sch (KiCad schematic)
At the start: 0 parts

Commit message: WIP power circuitry
Parts:
- added C1, C10, C3, C4, C7: 10u, Capacitor_SMD:C_0603_1608Metric_Pad1.08x0.95mm_HandSolder, symbol Device:C
- added C2, C5, C6, C8, C9: 1u, Capacitor_SMD:C_0402_1005Metric_Pad0.74x0.62mm_HandSolder, symbol Device:C
- added D1: BZX84C12LT1G, Package_TO_SOT_SMD:SOT-23, symbol Diode:BZX84Cxx
- added D2: SMAJ5.0CA, Diode_SMD:D_SMA, symbol Diode:SMAJ5.0CA
- added F1: MFU0603FF02000P500, Fuse:Fuse_0603_1608Metric_Pad1.05x0.95mm_HandSolder, symbol Device:Fuse
- added J2: S2B-PH-K-S, Connector_JST:JST_PH_S2B-PH-K_1x02_P2.00mm_Horizontal, symbol Connector:Conn_01x02_Pin
- added J3: M20-9750246, Connector_PinHeader_2.54mm:PinHeader_1x02_P2.54mm_Horizontal, symbol Connector:Conn_01x02_Pin
- added L1: LQH3NPZ2R2MMEL, kmm-pmask:IND_LQH3NPZ2R2MMEL, symbol Device:L
- added Q1: DMP3099L, Package_TO_SOT_SMD:SOT-23, symbol Transistor_FET:DMP3099L
- added R6: 100, Resistor_SMD:R_0402_1005Metric_Pad0.72x0.64mm_HandSolder, symbol Device:R
- added U2: TPS61202DRC, Package_SON:Texas_S-PVSON-N10_ThermalVias, symbol Regulator_Switching:TPS61202DRC
- added U3: AP2112K-3.3, Package_TO_SOT_SMD:SOT-23-5, symbol Regulator_Linear:AP2112K-3.3
- added U4: AP2112K-1.8, Package_TO_SOT_SMD:SOT-23-5, symbol Regulator_Linear:AP2112K-1.8
Connections:
- new net: D1.1 (A), Q1.1 (G), R6.1
- new net: D2.2 (A2), F1.2, Q1.3 (D)
- new net: C2.1, U2.1 (VAUX)
- new net: L1.2, U2.3 (L)
- new net +1.8V: C10.1, C9.1, U4.5 (VOUT)
- new net +3.3V: C6.1, C7.1, U3.5 (VOUT)
- new net +5V: C3.1, C4.1, U2.10 (FB), U2.2 (VOUT)
- new net BATT_IN: D1.3 (K), Q1.2 (S)
- new net BATT_RAW_P: F1.1, J2.1 (Pin_1), J3.1 (Pin_1)
- new net GND: C1.2, C10.2, C2.2, C3.2, C4.2, C5.2, C6.2, C7.2, C8.2, C9.2, D2.1 (A1), J2.2 (Pin_2), J3.2 (Pin_2), R6.2, U2.11 (PAD), U2.4 (PGND), U2.9 (GND), U3.2 (GND), U4.2 (GND)
- new net VS: C1.1, C5.1, C8.1, L1.1, U2.5 (VIN), U2.6 (EN), U2.7 (UVLO), U2.8 (PS), U3.1 (VIN), U3.3 (EN), U4.1 (VIN), U4.3 (EN)
Other:
- note added: "2.0 A 32 V Fast-Blow"
- note added: "2.2 µH 2.1 A"
- note added: "5.0 V_{R} 6.4 V_{C}"
- note added: "600 mA 1.8V LDO"
- note added: "600 mA 3.3V LDO"
- note added: "800 mA 5V Boost converter"
- note added: "Battery Input Protection"
- note added: "Battery Input Terminals"
- note added: "Recommended Supply Current per Power Rail, Slave Board"
- note added: "Reverse Polarity Protection"
- note added: "UVLO 250 mV"
- note added: "V_{Z} 12V (nom)"

Commit message: Initial draft of control board
Parts:
- added D3, D4, D5: LED GREEN, LED_SMD:LED_0603_1608Metric_Pad1.05x0.95mm_HandSolder, symbol Device:LED
- added R10, R11, R9: 10k, Resistor_SMD:R_0402_1005Metric_Pad0.72x0.64mm_HandSolder, symbol Device:R
- added R7, R8: 1M, Resistor_SMD:R_0402_1005Metric_Pad0.72x0.64mm_HandSolder, symbol Device:R
- added SW1: JS102011SAQN, Button_Switch_SMD:SW_SPDT_CK_JS102011SAQN, symbol Switch:SW_SPDT
- added TP10: +3.3V, TestPoint:TestPoint_Pad_D1.5mm, symbol Connector:TestPoint
- added TP11: +1.8V, TestPoint:TestPoint_Pad_D1.5mm, symbol Connector:TestPoint
- added TP12, TP13: GND, TestPoint:TestPoint_Pad_D1.5mm, symbol Connector:TestPoint
- added TP8: +BATT, TestPoint:TestPoint_Pad_D1.5mm, symbol Connector:TestPoint
- added TP9: +5V, TestPoint:TestPoint_Pad_D1.5mm, symbol Connector:TestPoint
Connections:
- net VS is gone; now on net +BATT: C1.1, C5.1, C8.1, L1.1, U2.5 (VIN), U2.6 (EN), U2.7 (UVLO), U2.8 (PS), U3.1 (VIN), U3.3 (EN), U4.1 (VIN), U4.3 (EN)
- net +1.8V: now also TP11.1
- net +3.3V: now also D5.2 (A), TP10.1
- net +5V: now also D4.2 (A), TP9.1
- net GND: now also R10.2, R11.2, R8.2, R9.2, SW1.1 (A), TP12.1, TP13.1; no longer R6.2
- net BATT_IN renamed +BATT
- net +BATT: now also D3.2 (A), R7.1, SW1.3 (C), TP8.1
- new net: D4.1 (K), R10.1
- new net: D3.1 (K), R9.1
- new net: D5.1 (K), R11.1
- new net BATT_SENSE: R7.2, R8.1
- new net PWR_ENABLE: R6.2, SW1.2 (B)
Other:
- note added: "+1.8 V rail is not included as most LED V_{f} is above 1.8 V"
- note added: "Battery Voltage Probe"
- note added: "Maximum Current Consumption per Power Rail, This Board"
- note added: "Power rail status indicators"
- note added: "See Datasheet section 11.2.3 for computation of peak current."
- note added: "Test Points"
- note added: "When PWR_ENABLE is shorted to +BATT, V_{GS} is 0 and power is disabled."
- title: (none) -> Power Management
- moved on the sheet: C1, C10, C2, C3, C4, C5, C6, C7, C8, C9, L1, U2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

Commit message: swap fuse for slow-blow
Parts:
- F1: value MFU0603FF02000P500 -> 0685T2000-01; footprint Fuse:Fuse_0603_1608Metric_Pad1.05x0.95mm_HandSolder -> Fuse:Fuse_1206_3216Metric_Pad1.42x1.75mm_HandSolder; Manufacturer P/N MFU0603FF02000P500 -> 0685T2000-01; Vendor P/N 749-MFU0603FF02000P500CT-ND -> 5923-0685T2000-01CT-ND
Changed lines of the file:
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@@
 		)
 	)
-	(text_box "A 1/2 Voltage divider to allow the MCU to approximate the current battery percentage."
+	(text_box "A 2:1 Voltage divider to allow the MCU to approximate the current battery percentage."
 		(exclude_from_sim no)
 		(at 204.47 64.77 0)
@@
 			)
 		)
-		(property "Value" "MFU0603FF02000P500"
+		(property "Value" "0685T2000-01"
 			(at 95.25 30.48 90)
 			(show_name no)
@@
 			)
 		)
-		(property "Footprint" "Fuse:Fuse_0603_1608Metric_Pad1.05x0.95mm_HandSolder"
+		(property "Footprint" "Fuse:Fuse_1206_3216Metric_Pad1.42x1.75mm_HandSolder"
 			(at 95.25 36.068 90)
 			(hide yes)
@@
 			)
 		)
-		(property "Datasheet" "https://www.vishay.com/docs/28747/mfuserie.pdf"
+		(property "Datasheet" "https://www.belfuse.com/media/datasheets/products/circuit-protection/ds-cp-c1t-series.pdf"
 			(at 95.25 34.29 0)
 			(hide yes)
@@
 			)
 		)
-		(property "Description" "2 A 32 V Fuse"
+		(property "Description" "FUSE BRD MNT 2A 63VAC 63VDC 1206"
 			(at 95.25 34.29 0)
 			(hide yes)
@@
 			)
 		)
-		(property "Manufacturer P/N" "MFU0603FF02000P500"
+		(property "Manufacturer P/N" "0685T2000-01"
 			(at 95.25 34.29 0)
 			(hide yes)
@@
 			)
 		)
-		(property "Vendor P/N" "749-MFU0603FF02000P500CT-ND"
+		(property "Vendor P/N" "5923-0685T2000-01CT-ND"
 			(at 95.25 34.29 0)
 			(hide yes)

Commit message: Initial PCB Layout
Parts:
- J2, J3: now not fitted
- TP10, TP11, TP12, TP13, TP8, TP9: footprint TestPoint:TestPoint_Pad_D1.5mm -> TestPoint:TestPoint_Pad_D1.0mm
Connections:
- net BATT_RAW_P: now also J3.2 (Pin_2); no longer J3.1 (Pin_1)
- net GND: now also J3.1 (Pin_1); no longer J3.2 (Pin_2)
Changed lines of the file:
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@@
 		)
 	)
+	(label "BATT_RAW_N"
+		(at 45.72 44.45 0)
+		(effects
+			(font
+				(size 1.27 1.27)
+			)
+			(justify left bottom)
+		)
+	)
 	(label "BATT_RAW_P"
 		(at 45.72 25.4 0)
@@
 		)
 	)
-	(label "BATT_RAW_N"
-		(at 45.72 46.99 0)
-		(effects
-			(font
-				(size 1.27 1.27)
-			)
-			(justify left bottom)
-		)
-	)
 	(label "PWR_ENABLE"
 		(at 180.34 46.99 0)
@@
 		)
 	)
-	(label "BATT_RAW_P"
-		(at 45.72 44.45 0)
+	(label "BATT_RAW_N"
+		(at 82.55 66.04 180)
 		(effects
 			(font
 				(size 1.27 1.27)
 			)
-			(justify left bottom)
+			(justify right bottom)
 		)
 	)
-	(label "BATT_RAW_N"
-		(at 82.55 66.04 180)
+	(label "BATT_RAW_P"
+		(at 45.72 46.99 0)
 		(effects
 			(font
 				(size 1.27 1.27)
 			)
-			(justify right bottom)
+			(justify left bottom)
 		)
 	)
@@
 			)
 		)
-		(property "Footprint" "TestPoint:TestPoint_Pad_D1.5mm"
+		(property "Footprint" "TestPoint:TestPoint_Pad_D1.0mm"
 			(at 261.62 31.75 0)
 			(hide yes)
@@
 		(on_board yes)
 		(in_pos_files yes)
-		(dnp no)
+		(dnp yes)
 		(property "Reference" "J2"
 			(at 36.83 25.4 0)
@@
 					(reference "J2")
 					(unit 1)
+					(variant
+						(name "2.54mm Battery Option")
+					)
+					(variant
+						(name "JST Battery Option")
+						(dnp no)
+					)
 				)
 			)
@@
 			)
 		)
-		(property "Footprint" "TestPoint:TestPoint_Pad_D1.5mm"
+		(property "Footprint" "TestPoint:TestPoint_Pad_D1.0mm"
 			(at 242.57 31.75 0)
 			(hide yes)
@@
 		(on_board yes)
 		(in_pos_files yes)
-		(dnp no)
+		(dnp yes)
 		(property "Reference" "J3"
 			(at 36.83 44.45 0)
@@
 					(reference "J3")
 					(unit 1)
+					(variant
+						(name "2.54mm Battery Option")
+						(dnp no)
+					)
+					(variant
+						(name "JST Battery Option")
+					)
 				)
 			)
@@
 			)
 		)
-		(property "Footprint" "TestPoint:TestPoint_Pad_D1.5mm"
+		(property "Footprint" "TestPoint:TestPoint_Pad_D1.0mm"
 			(at 252.73 53.34 0)
 			(hide yes)
@@
 			)
 		)
-		(property "Footprint" "TestPoint:TestPoint_Pad_D1.5mm"
+		(property "Footprint" "TestPoint:TestPoint_Pad_D1.0mm"
 			(at 255.27 31.75 0)
 			(hide yes)
@@
 			)
 		)
-		(property "Footprint" "TestPoint:TestPoint_Pad_D1.5mm"
+		(property "Footprint" "TestPoint:TestPoint_Pad_D1.0mm"
 			(at 248.92 31.75 0)
 			(hide yes)
@@
 			)
 		)
-		(property "Footprint" "TestPoint:TestPoint_Pad_D1.5mm"
+		(property "Footprint" "TestPoint:TestPoint_Pad_D1.0mm"
 			(at 259.08 53.34 0)
 			(hide yes)

Commit message: Add missing vendor part specifiers
Parts:
- Q1: Manufacturer P/N (none) -> DMP3099L-13; Vendor (none) -> DigiKey; Vendor P/N (none) -> DMP3099L-13DICT-ND
- U2: Manufacturer P/N (none) -> TPS61202DRCR; Vendor (none) -> DigiKey; Vendor P/N (none) -> 296-27462-1-ND
- U3: Manufacturer P/N (none) -> AP2112K-3.3TRG1; Vendor (none) -> DigiKey; Vendor P/N (none) -> AP2112K-3.3TRG1DICT-ND
- U4: Manufacturer P/N (none) -> AP2112K-1.8TRG1; Vendor (none) -> DigiKey; Vendor P/N (none) -> AP2112K-1.8TRG1DICT-ND
Changed lines of the file:
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@@
 			)
 		)
+		(property "Manufacturer P/N" "DMP3099L-13"
+			(at 133.35 36.83 0)
+			(hide yes)
+			(show_name no)
+			(do_not_autoplace no)
+			(effects
+				(font
+					(size 1.27 1.27)
+				)
+			)
+		)
+		(property "Vendor" "DigiKey"
+			(at 133.35 36.83 0)
+			(hide yes)
+			(show_name no)
+			(do_not_autoplace no)
+			(effects
+				(font
+					(size 1.27 1.27)
+				)
+			)
+		)
+		(property "Vendor P/N" "DMP3099L-13DICT-ND"
+			(at 133.35 36.83 0)
+			(hide yes)
+			(show_name no)
+			(do_not_autoplace no)
+			(effects
+				(font
+					(size 1.27 1.27)
+				)
+			)
+		)
 		(pin "2"
 		)
@@
 			)
 		)
+		(property "Manufacturer P/N" "TPS61202DRCR"
+			(at 63.5 109.22 0)
+			(hide yes)
+			(show_name no)
+			(do_not_autoplace no)
+			(effects
+				(font
+					(size 1.27 1.27)
+				)
+			)
+		)
+		(property "Vendor" "DigiKey"
+			(at 63.5 109.22 0)
+			(hide yes)
+			(show_name no)
+			(do_not_autoplace no)
+			(effects
+				(font
+					(size 1.27 1.27)
+				)
+			)
+		)
+		(property "Vendor P/N" "296-27462-1-ND"
+			(at 63.5 109.22 0)
+			(hide yes)
+			(show_name no)
+			(do_not_autoplace no)
+			(effects
+				(font
+					(size 1.27 1.27)
+				)
+			)
+		)
 		(pin "5"
 		)
@@
 			)
 		)
+		(property "Manufacturer P/N" "AP2112K-3.3TRG1"
+			(at 50.8 153.67 0)
+			(hide yes)
+			(show_name no)
+			(do_not_autoplace no)
+			(effects
+				(font
+					(size 1.27 1.27)
+				)
+			)
+		)
+		(property "Vendor" "DigiKey"
+			(at 50.8 153.67 0)
+			(hide yes)
+			(show_name no)
+			(do_not_autoplace no)
+			(effects
+				(font
+					(size 1.27 1.27)
+				)
+			)
+		)
+		(property "Vendor P/N" "AP2112K-3.3TRG1DICT-ND"
+			(at 50.8 153.67 0)
+			(hide yes)
+			(show_name no)
+			(do_not_autoplace no)
+			(effects
+				(font
+					(size 1.27 1.27)
+				)
+			)
+		)
 		(pin "4"
 		)
@@
 			(at 120.65 153.67 0)
 			(hide yes)
+			(show_name no)
+			(do_not_autoplace no)
+			(effects
+				(font
+					(size 1.27 1.27)
+				)
+			)
+		)
+		(property "Manufacturer P/N" "AP2112K-1.8TRG1"
+			(at 120.65 153.67 0)
+			(hide yes)
+			(show_name no)
+			(do_not_autoplace no)
+			(effects
+				(font
+					(size 1.27 1.27)
+				)
+			)
+		)
+		(property "Vendor" "DigiKey"
+			(at 120.65 153.67 0)
+			(hide yes)
+			(show_name no)
+			(do_not_autoplace no)
+			(effects
+				(font
+					(size 1.27 1.27)
+				)
+			)
+		)
+		(property "Vendor P/N" "AP2112K-1.8TRG1DICT-ND"
+			(at 120.65 153.67 0)
+			(hide yes)
