File: kmm-pmask-control/kmm-pmask-control.kicad_pcb (KiCad board)
At the start: 4 copper layers, 50 x 50 mm, 84 parts, among them J1 F31L-1A7H1-11030, J2 S2B-PH-K-S, J3 M20-9750246, J4 0472192001, J5 BD125-10-A-0305-0580-L-B, Q1 DMP3099L, SW1 JS102011SAQN, SW2 EVQ-P2402W, U1 PCA9517ADP, U2 TPS61202DRC, U3 AP2112K-3.3, U4 AP2112K-1.8, U5 MDBT50Q-P1MV2

Commit message: Add schematic PDF exports
Other:
- board text added: "All dimensions in mm"
